Commit message: add sensor

File: catkin_ws/src/zz_test/urdf/inc/camera.gazebo.xacro (robot description, xacro)
@@ -37,5 +37,5 @@
           <imageTopicName>image_raw</imageTopicName>
           <cameraInfoTopicName>camera_info</cameraInfoTopicName>
-          <frameName>wrist_3_link</frameName>
+          <frameName>camera_link</frameName>
           <hackBaseline>0.07</hackBaseline>
           <distortionK1>0.0</distortionK1>

File: catkin_ws/src/zz_test/urdf/inc/ur_macro.xacro (robot description, xacro)
@@ -317,11 +317,10 @@
     </joint>
     <!--- zz start  -->
+    <xacro:property name="camera_link" value="0.02" /> <!-- Size of square 'camera' box -->
     <joint name="camera_joint" type="fixed">
-      <axis xyz="0 1 0" />
-      <origin xyz="-0.02 0.0 0.055" rpy="0 0 0"/>
+      <origin xyz="0 0.05 0" rpy="0.0 ${-pi/2.0} ${-pi/2.0}" />
       <parent link="wrist_3_link"/>
       <child link="camera_link"/>
     </joint>
-    <xacro:property name="camera_link" value="0.05" /> <!-- Size of square 'camera' box -->
     <!-- Camera -->
     <link name="camera_link">
