Commit message: move ur description

File: catkin_ws/src/zz_test/urdf/inc/ur_macro.xacro (robot description, xacro)
@@ -320,5 +320,5 @@
       <axis xyz="0 1 0" />
       <origin xyz="-0.02 0.0 0.055" rpy="0 0 0"/>
-      <parent link="${prefix}wrist_3_link"/>
+      <parent link="wrist_3_link"/>
       <child link="camera_link"/>
     </joint>
@@ -329,11 +329,11 @@
         <origin xyz="0 0 0" rpy="0 0 0"/>
         <geometry>
-    <box size="${camera_link} ${camera_link} ${camera_link}"/>
-        </geometry>
-      </collision>
-      <visual>
-        <origin xyz="0 0 0" rpy="0 0 0"/>
-        <geometry>
-    <box size="${camera_link} ${camera_link} ${camera_link}"/>
+          <box size="${camera_link} ${camera_link} ${camera_link}"/>
+              </geometry>
+            </collision>
+            <visual>
+              <origin xyz="0 0 0" rpy="0 0 0"/>
+              <geometry>
+          <box size="${camera_link} ${camera_link} ${camera_link}"/>
         </geometry>
         <material name="green"/>
@@ -345,51 +345,6 @@
       </inertial>
     </link>
-    <gazebo reference="camera_link">
-      <mu1>0.2</mu1>
-      <mu2>0.2</mu2>
-      <material>Gazebo/Green</material>
-    </gazebo>
-    <gazebo reference="camera_link">
-      <sensor type="camera" name="camera1">
-        <update_rate>30.0</update_rate>
-        <camera name="head">
-          <horizontal_fov>1.3962634</horizontal_fov>
-          <image>
-            <width>800</width>
-            <height>800</height>
-            <format>R8G8B8</format>
-          </image>
-          <clip>
-            <near>0.02</near>
-            <far>300</far>
-          </clip>
-          <noise>
-            <type>gaussian</type>
-            <!-- Noise is sampled independently per pixel on each frame.
-                That pixel's noise value is added to each of its color
-                channels, which at that point lie in the range [0,1]. -->
-            <mean>0.0</mean>
-            <stddev>0.007</stddev>
-          </noise>
-        </camera>
-        <plugin name="camera_controller" filename="libgazebo_ros_camera.so">
-          <alwaysOn>true</alwaysOn>
-          <updateRate>0.0</updateRate>
-          <cameraName>rrbot/camera1</cameraName>
-          <imageTopicName>image_raw</imageTopicName>
-          <cameraInfoTopicName>camera_info</cameraInfoTopicName>
-          <frameName>wrist_3_link</frameName>
-          <hackBaseline>0.07</hackBaseline>
-          <distortionK1>0.0</distortionK1>
-          <distortionK2>0.0</distortionK2>
-          <distortionK3>0.0</distortionK3>
-          <distortionT1>0.0</distortionT1>
-          <distortionT2>0.0</distortionT2>
-        </plugin>
-        <always_on>1</always_on>
-        <visualize>true</visualize>
-      </sensor>
-    </gazebo>
     <!--- zz end  -->
   </xacro:macro>
+  <xacro:include filename="$(find zz_test)/urdf/inc/camera.gazebo.xacro" />
 </robot>

Commit message: add cylinder to urdf

File: catkin_ws/src/zz_test/urdf/inc/ur_macro.xacro (robot description, xacro)
@@ -344,4 +344,31 @@
       </inertial>
     </link>
+    <joint name="ee_joint" type="fixed">
+      <origin xyz="0 0 0" />
+      <parent link="wrist_3_link"/>
+      <child link="ee_link"/>
+    </joint>
+    <link name="ee_link">
+      <collision>
+        <origin xyz="0 0 0.075" rpy="0 0 0"/>
+        <geometry>
+          <cylinder length="0.14" radius="0.03"/>
+        </geometry>
+      </collision>
+      <visual>
+        <origin xyz="0 0 0.075" rpy="0 0 0"/>
+        <geometry>
+          <cylinder length="0.14" radius="0.03"/>
+        </geometry>
+      </visual>
+      <inertial>
+        <origin xyz="0 0 0.075" rpy="0 0 0"/>
+        <mass value="0.00001"/>
+        <inertia
+          ixx="0.00001" ixy="0.0" ixz="0.0"
+          iyy="0.00001" iyz="0.0"
+          izz="0.00001"/>
+      </inertial>
+    </link>
     <!--- zz end  -->
   </xacro:macro>

Commit message: end effector

File: catkin_ws/src/zz_test/urdf/inc/ur_macro.xacro (robot description, xacro)
@@ -317,11 +317,12 @@
     </joint>
     <!--- zz start  -->
-    <xacro:property name="camera_link" value="0.02" /> <!-- Size of square 'camera' box -->
+      <!-- Camera -->
+    <!--
+      <xacro:property name="camera_link" value="0.02" />
     <joint name="camera_joint" type="fixed">
-      <origin xyz="0 0.05 0" rpy="0.0 ${-pi/2.0} ${-pi/2.0}" />
+      <origin xyz="0 0.07 0" rpy="0.0 ${-pi/2.0} ${-pi/2.0}" />
       <parent link="wrist_3_link"/>
       <child link="camera_link"/>
     </joint>
-    <!-- Camera -->
     <link name="camera_link">
       <collision>
@@ -343,25 +344,27 @@
         <inertia ixx="1e-6" ixy="0" ixz="0" iyy="1e-6" iyz="0" izz="1e-6" />
       </inertial>
-    </link>
-    <joint name="ee_joint" type="fixed">
+    </link> -->
+    <!-- <xacro:include filename="$(find zz_test)/urdf/inc/camera.gazebo.xacro" /> -->
+    <!-- end effector -->
+    <joint name="eelink_joint" type="fixed">
       <origin xyz="0 0 0" />
       <parent link="wrist_3_link"/>
-      <child link="ee_link"/>
-    </joint>
-    <link name="ee_link">
-      <collision>
-        <origin xyz="0 0 0.075" rpy="0 0 0"/>
-        <geometry>
-          <cylinder length="0.14" radius="0.03"/>
-        </geometry>
-      </collision>
-      <visual>
-        <origin xyz="0 0 0.075" rpy="0 0 0"/>
-        <geometry>
-          <cylinder length="0.14" radius="0.03"/>
+      <child link="eelink_link"/>
+    </joint>
+    <link name="eelink_link">
+      <collision>
+        <origin xyz="0 0 0.026" rpy="0 0 0"/>
+        <geometry>
+          <cylinder length="0.05" radius="0.03"/>
+        </geometry>
+      </collision>
+      <visual>
+        <origin xyz="0 0 0.026" rpy="0 0 0"/>
+        <geometry>
+          <cylinder length="0.05" radius="0.03"/>
         </geometry>
       </visual>
       <inertial>
-        <origin xyz="0 0 0.075" rpy="0 0 0"/>
+        <origin xyz="0 0 0.026" rpy="0 0 0"/>
         <mass value="0.00001"/>
         <inertia
@@ -371,6 +374,59 @@
       </inertial>
     </link>
+    <joint name="ee_joint" type="fixed">
+      <origin xyz="0 0 0" />
+      <parent link="wrist_3_link"/>
+      <child link="ee_link"/>
+    </joint>
+    <link name="ee_link">
+      <collision>
+        <origin xyz="0 0 0.086" rpy="0 0 0"/>
+        <geometry>
+          <cylinder length="0.07" radius="0.05"/>
+        </geometry>
+      </collision>
+      <visual>
+        <origin xyz="0 0 0.086" rpy="0 0 0"/>
+        <geometry>
+          <cylinder length="0.07" radius="0.05"/>
+        </geometry>
+      </visual>
+      <inertial>
+        <origin xyz="0 0 0.086" rpy="0 0 0"/>
+        <mass value="0.00001"/>
+        <inertia
+          ixx="0.00001" ixy="0.0" ixz="0.0"
+          iyy="0.00001" iyz="0.0"
+          izz="0.00001"/>
+      </inertial>
+    </link>
+    <joint name="touch_joint" type="fixed">
+      <origin xyz="0 0 0" />
+      <parent link="wrist_3_link"/>
+      <child link="touch_link"/>
+    </joint>
+    <link name="touch_link">
+      <collision>
+        <origin xyz="0 0 0.146" rpy="0 0 0"/>
+        <geometry>
+          <cylinder length="0.04" radius="0.03"/>
+        </geometry>
+      </collision>
+      <visual>
+        <origin xyz="0 0 0.146" rpy="0 0 0"/>
+        <geometry>
+          <cylinder length="0.04" radius="0.03"/>
+        </geometry>
+      </visual>
+      <inertial>
+        <origin xyz="0 0 0.146" rpy="0 0 0"/>
+        <mass value="0.00001"/>
+        <inertia
+          ixx="0.00001" ixy="0.0" ixz="0.0"
+          iyy="0.00001" iyz="0.0"
+          izz="0.00001"/>
+      </inertial>
+    </link>
     <!--- zz end  -->
   </xacro:macro>
-  <xacro:include filename="$(find zz_test)/urdf/inc/camera.gazebo.xacro" />
 </robot>

Commit message: avoid hit table

File: catkin_ws/src/zz_test/urdf/inc/ur_macro.xacro (robot description, xacro)
@@ -319,5 +319,5 @@
     <xacro:property name="camera_link" value="0.02" /> <!-- Size of square 'camera' box -->
     <joint name="camera_joint" type="fixed">
-      <origin xyz="0 0.05 0" rpy="0.0 ${-pi/2.0} ${-pi/2.0}" />
+      <origin xyz="0 0.06 0.05" rpy="0.0 ${-pi/2.0} ${-pi/2.0}" />
       <parent link="wrist_3_link"/>
       <child link="camera_link"/>
@@ -351,17 +351,17 @@
     <link name="ee_link">
       <collision>
-        <origin xyz="0 0 0.075" rpy="0 0 0"/>
-        <geometry>
-          <cylinder length="0.14" radius="0.03"/>
-        </geometry>
-      </collision>
-      <visual>
-        <origin xyz="0 0 0.075" rpy="0 0 0"/>
-        <geometry>
-          <cylinder length="0.14" radius="0.03"/>
+        <origin xyz="0 0 0.065" rpy="0 0 0"/>
+        <geometry>
+          <cylinder length="0.12" radius="0.05"/>
+        </geometry>
+      </collision>
+      <visual>
+        <origin xyz="0 0 0.065" rpy="0 0 0"/>
+        <geometry>
+          <cylinder length="0.12" radius="0.05"/>
         </geometry>
       </visual>
       <inertial>
-        <origin xyz="0 0 0.075" rpy="0 0 0"/>
+        <origin xyz="0 0 0.065" rpy="0 0 0"/>
         <mass value="0.00001"/>
         <inertia

Commit message: radius 0.6

File: catkin_ws/src/zz_test/urdf/inc/ur_macro.xacro (robot description, xacro)
@@ -319,5 +319,5 @@
     <xacro:property name="camera_link" value="0.02" /> <!-- Size of square 'camera' box -->
     <joint name="camera_joint" type="fixed">
-      <origin xyz="0 0.06 0.05" rpy="0.0 ${-pi/2.0} ${-pi/2.0}" />
+      <origin xyz="0 0.07 0.05" rpy="0.0 ${-pi/2.0} ${-pi/2.0}" />
       <parent link="wrist_3_link"/>
       <child link="camera_link"/>
@@ -353,5 +353,5 @@
         <origin xyz="0 0 0.065" rpy="0 0 0"/>
         <geometry>
-          <cylinder length="0.12" radius="0.05"/>
+          <cylinder length="0.12" radius="0.06"/>
         </geometry>
       </collision>
@@ -359,5 +359,5 @@
         <origin xyz="0 0 0.065" rpy="0 0 0"/>
         <geometry>
-          <cylinder length="0.12" radius="0.05"/>
+          <cylinder length="0.12" radius="0.06"/>
         </geometry>
       </visual>

Commit message: move camera

File: catkin_ws/src/zz_test/urdf/inc/ur_macro.xacro (robot description, xacro)
@@ -319,5 +319,5 @@
     <xacro:property name="camera_link" value="0.02" /> <!-- Size of square 'camera' box -->
     <joint name="camera_joint" type="fixed">
-      <origin xyz="0 0.07 0.05" rpy="0.0 ${-pi/2.0} ${-pi/2.0}" />
+      <origin xyz="0 0.07 0.07" rpy="0.0 ${-pi/2.0} ${-pi/2.0}" />
       <parent link="wrist_3_link"/>
       <child link="camera_link"/>
